File: hardware/Gateway_Schematic_V3/Schematic_V2_backup/Gateway_Schematic_V3.kicad_pcb (KiCad board)
At the start: 2 copper layers, 193.2 x 111.3 mm, 197 parts, among them IC1 RTC_DS3231M, IC2 SIM7600CE-H, J1 USB_C_Receptacle_USB2.0_14P, J10 ANT_LTE, J11 ANT_LTE, J12 ANT_LTE, J14 SIM7100-6pin-socket-smd, J17 HR911105A, J2 Conn_01x04_Pin, J3 Screw_Terminal_01x03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

Commit message: Update PCB Layout for Gateway (24/3/2026)
Parts:
- added CLK0: ~, IVS_NEW_FOOTPRINT:TestPoint_throughtHole_D1.0mm, F.Cu at (245.6, 158.8)
- added CS0: ~, IVS_NEW_FOOTPRINT:TestPoint_throughtHole_D1.0mm, F.Cu at (245.6, 166.4)
- added CS1: TestPoint, IVS_NEW_FOOTPRINT:TestPoint_throughtHole_D1.0mm, F.Cu at (317.0, 202.3)
- added ESP_RX1: TestPoint, IVS_NEW_FOOTPRINT:TestPoint_throughtHole_D1.0mm, F.Cu at (301.1, 191.6)
- added ESP_SCL0: TestPoint, IVS_NEW_FOOTPRINT:TestPoint_throughtHole_D1.0mm, F.Cu at (248.3, 210.2)
- added ESP_SDA0: TestPoint, IVS_NEW_FOOTPRINT:TestPoint_throughtHole_D1.0mm, F.Cu at (248.3, 212.7)
- added ESP_TX1: TestPoint, IVS_NEW_FOOTPRINT:TestPoint_throughtHole_D1.0mm, F.Cu at (301.1, 189.1)
- added GND0: TestPoint, IVS_NEW_FOOTPRINT:TestPoint_throughtHole_D1.0mm, F.Cu at (245.6, 169.0)
- added GND0: TestPoint, IVS_NEW_FOOTPRINT:TestPoint_throughtHole_D1.0mm, F.Cu at (248.3, 215.3)
- added GND0: TestPoint, IVS_NEW_FOOTPRINT:TestPoint_throughtHole_D1.0mm, F.Cu at (295.0, 194.1)
- added GND1: TestPoint, IVS_NEW_FOOTPRINT:TestPoint_throughtHole_D1.0mm, F.Cu at (301.1, 194.1)
- added GND1: TestPoint, IVS_NEW_FOOTPRINT:TestPoint_throughtHole_D1.0mm, F.Cu at (319.5, 202.3)
- added MISO0: ~, IVS_NEW_FOOTPRINT:TestPoint_throughtHole_D1.0mm, F.Cu at (245.6, 163.9)
- added MISO1: TestPoint, IVS_NEW_FOOTPRINT:TestPoint_throughtHole_D1.0mm, F.Cu at (314.4, 202.3)
- added MOSI0: ~, IVS_NEW_FOOTPRINT:TestPoint_throughtHole_D1.0mm, F.Cu at (245.6, 161.4)
- added MOSI1: TestPoint, IVS_NEW_FOOTPRINT:TestPoint_throughtHole_D1.0mm, F.Cu at (311.9, 202.3)
- added RX0: ~, IVS_NEW_FOOTPRINT:TestPoint_throughtHole_D1.0mm, F.Cu at (295.0, 191.6)
- added SCK1: TestPoint, IVS_NEW_FOOTPRINT:TestPoint_throughtHole_D1.0mm, F.Cu at (309.4, 202.3)
- added TX0: ~, IVS_NEW_FOOTPRINT:TestPoint_throughtHole_D1.0mm, F.Cu at (295.0, 189.1)
- +1.8V1: renamed from +1.8V; footprint TestPoint:TestPoint_Pad_D1.0mm -> IVS_NEW_FOOTPRINT:TestPoint_throughtHole_D1.0mm
- PWRKEY1: renamed from PWRKEY; footprint TestPoint:TestPoint_Pad_D1.0mm -> IVS_NEW_FOOTPRINT:TestPoint_throughtHole_D1.0mm
- RESET1: renamed from RESET; footprint TestPoint:TestPoint_Pad_D1.0mm -> IVS_NEW_FOOTPRINT:TestPoint_throughtHole_D1.0mm
- RXD1: renamed from RXD; footprint TestPoint:TestPoint_Pad_D1.0mm -> IVS_NEW_FOOTPRINT:TestPoint_throughtHole_D1.0mm
- TP1: renamed from +5V; footprint TestPoint:TestPoint_Pad_D1.0mm -> IVS_NEW_FOOTPRINT:TestPoint_throughtHole_D1.0mm
- TP13: renamed from +4V; footprint TestPoint:TestPoint_Pad_D1.0mm -> IVS_NEW_FOOTPRINT:TestPoint_throughtHole_D1.0mm
- TXD1: renamed from TXD; footprint TestPoint:TestPoint_Pad_D1.0mm -> IVS_NEW_FOOTPRINT:TestPoint_throughtHole_D1.0mm
- VDD_AUX1: renamed from VDD_AUX; footprint TestPoint:TestPoint_Pad_D1.0mm -> IVS_NEW_FOOTPRINT:TestPoint_throughtHole_D1.0mm
- renumbered LED1 to LE1, LED2 to LE2
Routing:
- net /ESP32-S3/ESP_ETH.CLK: track 80.0 -> 102.1 mm, vias 0 -> 1
- net /ESP32-S3/ESP_ETH_CS: track 82.6 -> 93.5 mm, vias 0 -> 1
- net /ESP32-S3/ESP_HMI_RX: track 80.0 -> 90.4 mm
- net /ESP32-S3/LORA.MOSI: track 51.9 -> 61.9 mm, vias 0 -> 2
- net /ESP32-S3/ESP_ETH.MISO: track 77.2 -> 86.1 mm, vias 0 -> 1
- net /ESP32-S3/ESP_ETH.MOSI: track 75.2 -> 83.7 mm, vias 0 -> 1
- net /ESP32-S3/LORA.SCK: track 45.7 -> 53.3 mm
- net /ESP32-S3/UART1_RX: track 38.3 -> 45.7 mm
- net /ESP32-S3/LORA.CS: track 54.6 -> 60.7 mm
- net GND: track 279.3 -> 285.2 mm
- net /ESP32-S3/LORA.MISO: track 49.0 -> 54.6 mm
- net /ESP32-S3/UART1_TX: track 32.9 -> 38.1 mm
- net /ESP32-S3/ESP.SDA: track 106.4 -> 111.7 mm
- net /ESP32-S3/ESP_HMI_TX: track 85.2 -> 89.0 mm
- net /ESP32-S3/ESP.SCL: track 94.8 -> 98.0 mm
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Other:
- board text added: "(HMI)"
- board text added: "(SIM)"
