File: hardware/Gateway_Schematic_V3/Schematic_V2_backup/untitled.kicad_sch (KiCad schematic)
At the start: 58 parts, among them IC2 SIM7600CE-H, J10 ANT_LTE, J11 ANT_LTE, J12 ANT_LTE, J14 SIM7100-6pin-socket-smd, Q1 MMBT3904, Q2 BC817, Q3 BC817, Q4 BC817, Q8 MMBT3904

Commit message: Update PCB Layout for Gateway (24/3/2026)
Parts:
- removed C3: 100nF, Capacitor_SMD:C_0603_1608Metric, symbol Device:C
- removed C4: 10uF, Capacitor_SMD:C_0603_1608Metric, symbol Device:C
- removed C600, C601: 100nF, IVS_FOOTPRINTS:C_0603, symbol Device:C
- removed D60, D61: PSD12C, Diode_SMD:D_SOD-323, symbol Diode:ESD9B3.3ST5G
- removed Q4: BC817, Package_TO_SOT_SMD:SOT-23, symbol Transistor_BJT:BC817
- added J13, J19: 20279-001E-03, Library_gateway:IPEX, symbol New_Library:20279-001E-03
- added Q6: BC807, Package_TO_SOT_SMD:SOT-23, symbol Transistor_BJT:BC807
- added R36, R38: 2K2, Resistor_SMD:R_0603_1608Metric, symbol Device:R
- added TP14, TP5, TP9: ~, TestPoint:TestPoint_Pad_D1.0mm, symbol Connector:TestPoint
- C250, C251, C253: footprint IVS_FOOTPRINTS:C_0603 -> (none)
- D4: footprint GATEWAY_LIB:SC70-6 -> Library_gateway:SC70-6
- IC2: footprint GATEWAY_LIB:SIM7600 -> Library_gateway:SIM7600
- J10, J11, J12: footprint IVS_NEW_FOOTPRINT:Conn_IPEX_ANT -> Connector_Coaxial:SMA_BAT_Wireless_BWSMA-KWE-Z001
- J14: footprint GATEWAY_LIB:GCT_SIM7100-6-socket-smd -> Library_gateway:GCT_SIM7100-6-socket-smd
- R250: footprint IVS_FOOTPRINTS:R_0603 -> (none)
Connections:
- net GND: now also J13.2, J13.3, J19.2, J19.3, Q6.2 (E)
- net UART1_RX: now also TP14.1
- net VDD_1_8V: now also R36.2, R38.2
- net at C45.2, IC2.82 (MAIN_ANT), R47.2: now also J13.1
- net at C43.2, IC2.59 (AUX_ANT), R44.2: now also J19.1
- net at R60.2, R61.1: now also Q6.1 (B)
- net I2C2_SCL: now reaches IC2.55 (SCL)
- net I2C2_SCL: now also R38.1, TP9.1
- net I2C2_SDA: now reaches IC2.56 (SDA)
- net I2C2_SDA: now also R36.1, TP5.1
- net at R62.1: now also Q6.3 (C)
- net ESP_PWRKEY renamed ST_PWRKEY
- net ESP_RST renamed ST_RST
- no-connect marks 48 -> 46
Other:
- note added: "BC807 LÀ PNP ==> CẦN DÙNG NPN THÌ MỚI ĐÚNG NGUYÊN LÝ"
- note added: "nếu không chắc thì nhớ bật chân scl, sda xuống 0"
- note removed: "Tụ và ESD: Tụ xử lý nhiễu nhỏ, giúp tín hiệu mượt hơn ESD xử lý sốc lớn khi tín hiệu hay đổi đột ngột, chống sốc tĩnh điện"
- moved on the sheet: C250, C251, C253, C41, C42, C43, C44, C45, C46, C47, C48, C49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
