File: hardware/Gateway_Schematic_V3/Gateway_Schematic_V3.kicad_pcb (KiCad board)
At the start: 2 copper layers, 193.2 x 111.3 mm, 216 parts, among them IC1 RTC_DS3231M, IC2 SIM7600CE-H, J1 USB_C_Receptacle_USB2.0_14P, J10 ANT_LTE, J11 ANT_LTE, J12 ANT_LTE, J14 SIM7100-6pin-socket-smd, J2 Conn_01x04_Pin, J3 Screw_Terminal_01x03, J5 MiSD-PP-9P-V1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

Commit message: Update Solder Bridge for 3v3 and 4v
Parts:
- added JP1: SolderJumper_2_Open, IVS_NEW_FOOTPRINT:SolderJumper-2_P1.3mm_Open_RoundedPad1.0x1.5mm, F.Cu at (212.1, 230.5)
- added JP2: SolderJumper_2_Open, IVS_NEW_FOOTPRINT:SolderJumper-2_P1.3mm_Open_RoundedPad1.0x1.5mm, F.Cu at (216.5, 228.0)
- added U12: Ipex, IVS_NEW_FOOTPRINT:Conn_IPEX_ANT, F.Cu at (1.82, 2.31)
- moved +4V 5.41 mm to (213.9, 224.6)
- moved +5V 0.07 mm to (219.2, 233.1)
- renumbered +3V3 to +5V, ETHERNET to J17, TX0 to TP2, RX0 to TP3
Connections:
- +4V pad 1: +4V -> /Khối nguồn/4v_SIM
- C1 pad 2: +3.3V -> +3V3
- C2 pad 2: +3.3V -> +3V3
- C20 pad 1: +3.3V -> +3V3
- C21 pad 1: +3.3V -> +3V3
- C251 pad 1: +3.3V -> +3V3
- C27 pad 2: +3.3V -> +3V3
- C35 pad 1: +3.3V -> +3V3
- C36 pad 1: +3.3V -> +3V3
- C57 pad 1: +3.3V -> +3V3
- C58 pad 1: +3.3V -> +3V3
- C66 pad 1: +3.3V -> +3V3
- C83 pad 1: +4V -> /Khối nguồn/4v_SIM
- C84 pad 1: +4V -> /Khối nguồn/4v_SIM
- C85 pad 1: +4V -> /Khối nguồn/4v_SIM
- FB1 pad 2: +3.3V -> +3V3
- IC1 pad 2: +3.3V -> +3V3
- J17 pad 12: +3.3V -> +3V3
- J17 pad 9: +3.3V -> +3V3
- J5 pad 4: +3.3V -> +3V3
- J6 pad 2: +3.3V -> +3V3
- L2 pad 2: +4V -> /Khối nguồn/4v_SIM
- LE5 pad 1: +3.3V -> +3V3
- R1 pad 1: +3.3V -> +3V3
- R101 pad 2: +4V -> /Khối nguồn/4v_SIM
- R102 pad 1: +4V -> /Khối nguồn/4v_SIM
- R14 pad 1: +3.3V -> +3V3
- R17 pad 1: +3.3V -> +3V3
- R18 pad 1: +3.3V -> +3V3
- R19 pad 1: +3.3V -> +3V3
- R20 pad 1: +3.3V -> +3V3
- R21 pad 1: +3.3V -> +3V3
- R24 pad 1: +3.3V -> +3V3
- R25 pad 1: +3.3V -> +3V3
- R29 pad 1: +3.3V -> +3V3
- R33 pad 1: +3.3V -> +3V3
- R34 pad 1: +3.3V -> +3V3
- R49 pad 2: +3.3V -> +3V3
- R654 pad 2: +3.3V -> +3V3
- R66 pad 1: +3.3V -> +3V3
- R67 pad 1: +3.3V -> +3V3
- R68 pad 1: +3.3V -> +3V3
- R71 pad 1: +3.3V -> +3V3
- R72 pad 1: +3.3V -> +3V3
- U1 pad 2: +3.3V -> +3V3
- U8 pad 3: +3.3V -> +3V3
- U9 pad 28: +3.3V -> +3V3
Routing:
- net +3.3V: track 634.1 -> 41.6 mm, vias 24 -> 2
- net +3V3: track 0.00 -> 591.3 mm, vias 0 -> 22
- net /Khối nguồn/4v_SIM: track 0.00 -> 70.7 mm, vias 0 -> 2
- net +4V: track 178.1 -> 108.7 mm, vias 4 -> 2

Commit message: Update PCB Layout for Gateway (add test point and change button)
Parts:
- removed U12: Ipex, IVS_NEW_FOOTPRINT:Conn_IPEX_ANT
- SW1, SW2: footprint IVS_FOOTPRINTS:SW_SPST_PTS810 -> Button_Switch_SMD:SW_SPST_B3U-1000P
- moved SW1 0.51 mm to (306.9, 151.8)
- moved SW2 0.36 mm to (271.7, 151.8), turned to -90 degrees
- renumbered +5V to TP1, +4V to TP13
Routing:
- net GND: track 285.2 -> 276.4 mm
- net /ESP32-S3/BOOT: track 51.0 -> 47.1 mm
- net /ESP32-S3/RST: track 53.6 -> 49.7 mm
