File: hardware/Gateway_Schematic_V3/Gateway_Schematic_V3.kicad_pcb (KiCad board)
At the start: 2 copper layers, 193.2 x 111.3 mm, 219 parts, among them IC1 RTC_DS3231M, IC2 SIM7600CE-H, J1 USB_C_Receptacle_USB2.0_14P, J10 ANT_LTE, J11 ANT_LTE, J12 ANT_LTE, J14 SIM7100-6pin-socket-smd, J17 HR911105A, J2 Conn_01x04_Pin, J3 Screw_Terminal_01x03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

Commit message: feat: Second review
Thay đổi kích thước chữ từ 1mm thành 0.8mm của các linh kiện - resize 1mm text size to 0.8mm
change direction of text footprint across placement direction
Note: Nhớ thay đổi footprint của nút nhấn
Thay đổi vị trí chữ để không bị chồng lấn với via
Parts:
- removed U12: Ipex, IVS_NEW_FOOTPRINT:Conn_IPEX_ANT
- SW1, SW2: footprint IVS_FOOTPRINTS:SW_SPST_PTS810 -> Button_Switch_SMD:SW_SPST_B3U-1000P
- moved SW1 0.51 mm to (306.9, 151.8)
- moved SW2 0.36 mm to (271.7, 151.8), turned to -90 degrees
- renumbered +5V to TP1, +4V to TP13
Routing:
- net GND: track 285.2 -> 276.5 mm
- net /ESP32-S3/BOOT: track 51.0 -> 47.1 mm
- net /ESP32-S3/RST: track 53.6 -> 49.7 mm
